File: Hardware/Main-board/Bad Thing of the Edge Keyboard.kicad_pcb (KiCad board)
At the start: 2 copper layers, 118.6 x 145.8 mm, 61 parts, among them J1 Conn_01x01_Pin, J2 Conn_01x01_Pin, J3 Conn_01x01_Pin, J4 Conn_01x01_Pin, J5 Conn_01x01_Pin, J6 Conn_01x01_Pin, Q1 BSS138, Q2 BSS138, Q3 BSS138, Q4 BSS138, SW1 SW_Push, SW10 SW_Push, SW11 SW_Push, SW12 SW_Push, SW13 SW_Push, SW14 SW_Push, SW15 SW_Push, SW16 SW_Push, SW17 SW_Push, SW18 SW_Push, SW19 SW_Push, SW2 SW_Push, SW20 SW_Push, SW3 SW_Push, SW4 SW_Push, SW5 SW_Push, SW6 SW_Push, SW7 SW_Push, SW8 SW_Push, SW9 SW_Push, U1 Pico, m1 OSHW-Logo2_14.6x12mm_SilkScre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, m2 KiCad-Logo2_5mm_SilkScreen

Commit message: Main board revision 3
Connections:
- Q2 pad 1: unconnected-(Q2-G-Pad1) -> Net-(Q2-G)
- R5 pad 2: Net-(R5-Pad2) -> Net-(Q2-G)
- R6 pad 1: Net-(R5-Pad2) -> Net-(Q2-G)
Routing:
- net Net-(Q2-G): track 0.00 -> 7.53 mm
- net Net-(R5-Pad2): track 3.56 -> 0.00 mm
- net GNDREF: vias 89 -> 94
Other:
- board text added: "3.0"
- board text removed: "2.0"
