File: Hardware/Main-board/Bad Thing of the Edge Keyboard.kicad_sch (KiCad schematic)
At the start: 59 parts, among them J1 Conn_01x01_Pin, J2 Conn_01x01_Pin, J3 Conn_01x01_Pin, J4 Conn_01x01_Pin, J5 Conn_01x01_Pin, J6 Conn_01x01_Pin, Q1 BSS138, Q2 BSS138, Q3 BSS138, Q4 BSS138, SW1 SW_Push, SW10 SW_Push, SW11 SW_Push, SW12 SW_Push, SW13 SW_Push, SW14 SW_Push, SW15 SW_Push, SW16 SW_Push, SW17 SW_Push, SW18 SW_Push, SW19 SW_Push, SW2 SW_Push, SW20 SW_Push, SW3 SW_Push, SW4 SW_Push, SW5 SW_Push, SW6 SW_Push, SW7 SW_Push, SW8 SW_Push, SW9 SW_Push, U1 Pico

Commit message: Main board revision 3
Connections:
- net at R5.2, R6.1: now also Q2.1 (G)
Other:
- note added: "3.0"
Changed lines of the file:
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@@
   (junction (at 48.26 185.42) (diameter 0) (color 0 0 0 0)
+  )
+  (junction (at 72.39 175.26) (diameter 0) (color 0 0 0 0)
   )
   (junction (at 87.63 147.32) (diameter 0) (color 0 0 0 0)
@@
     (stroke (width 0) (type default))
   )
+  (wire (pts (xy 72.39 175.26) (xy 72.39 176.53))
+    (stroke (width 0) (type default))
+  )
   (wire (pts (xy 87.63 168.91) (xy 87.63 170.18))
     (stroke (width 0) (type default))
@@
     (stroke (width 0) (type default))
   )
-  (wire (pts (xy 72.39 171.45) (xy 72.39 176.53))
+  (wire (pts (xy 72.39 171.45) (xy 72.39 175.26))
     (stroke (width 0) (type default))
   )
@@
   )
   (wire (pts (xy 160.02 113.03) (xy 148.59 113.03))
+    (stroke (width 0) (type default))
+  )
+  (wire (pts (xy 69.85 175.26) (xy 72.39 175.26))
     (stroke (width 0) (type default))
   )
@@
     (effects (font (face "Arial") (size 15 15) (thickness 1) bold (color 0 0 0 1)) (justify left bottom))
   )
+  (text "3.0" (at 269.24 194.31 0)
+    (effects (font (size 1.27 1.27)) (justify left bottom))
+  )
   (text "EDGE" (at 233.68 63.5 0)
