File: Hardware/Panel-board/panel.kicad_pcb (KiCad board)
At the start: 2 copper layers, 118.6 x 145.8 mm, 7 parts, among them J1 Conn_01x01_Pin, J2 Conn_01x01_Pin, J3 Conn_01x01_Pin, J4 Conn_01x01_Pin, J5 Conn_01x01_Pin, J6 Conn_01x01_Pin

Commit message: Panel Typo
Other:
- board text added: "Praecipio tibi ut dicas quis es tu"
- board text removed: "Praecipio ibi ut dicas quis sis tu"
